File: PCB/uranus-pocket-tbc.kicad_pcb (KiCad board)
At the start: 2 copper layers, 200 x 30 mm, 10 parts, among them U1 ST25DV04KC-IE8S3

Commit message: update schematic, oops
Routing:
- net (no net): track 27.5 -> 0.00 mm
Changed lines of the file:
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@@
-	)
-	(segment
-		(start 237.5 84.25)
-		(end 240 84.25)
-		(width 1.016)
-		(layer "B.Cu")
-		(net "")
-	)
-	(segment
-		(start 237.5 76.75)
-		(end 240 76.75)
-		(width 0.2032)
-		(layer "B.Cu")
-		(net "")
-	)
-	(segment
-		(start 237.5 83)
-		(end 240 83)
-		(width 0.762)
-		(layer "B.Cu")
-		(net "")
-	)
-	(segment
-		(start 237.5 74.25)
-		(end 240 74.25)
-		(width 0.127)
-		(layer "B.Cu")
-		(net "")
-	)
-	(segment
-		(start 237.5 80.5)
-		(end 240 80.5)
-		(width 0.381)
-		(layer "B.Cu")
-		(net "")
-	)
-	(segment
-		(start 237.5 79.25)
-		(end 240 79.25)
-		(width 0.3048)
-		(layer "B.Cu")
-		(net "")
-	)
-	(segment
-		(start 237.5 75.5)
-		(end 240 75.5)
-		(width 0.1524)
-		(layer "B.Cu")
-		(net "")
-	)
-	(segment
-		(start 237.5 87.5)
-		(end 240 87.5)
-		(width 1.27)
-		(layer "B.Cu")
-		(net "")
-	)
-	(segment
-		(start 237.5 81.75)
-		(end 240 81.75)
-		(width 0.508)
-		(layer "B.Cu")
-		(net "")
-	)
-	(segment
-		(start 237.51 85.5472)
-		(end 240.01 85.5472)
-		(width 1.27)
-		(layer "B.Cu")
-		(net "")
-	)
-	(segment
-		(start 237.5 78)
-		(end 240 78)
-		(width 0.254)
-		(layer "B.Cu")
-		(net "")
 	)
 	(segment
@@
 	)
 	(zone
-		(net "Net-(U1-AC0)")
-		(layer "F.Cu")
-		(hatch none 0.1)
-		(priority 30001)
-		(attr
-			(teardrop
-				(type padvia)
-			)
-		)
-		(connect_pads yes
-			(clearance 0)
-		)
-		(min_thickness 0.0254)
-		(fill yes
-			(island_removal_mode 1)
-		)
-		(polygon
-			(pts
-				(xy 52.118353 81.612158) (xy 52.297958 81.432553) (xy 52.009499 81.107101) (xy 51.889251 81.203451)
-				(xy 51.941246 81.472044)
-			)
-		)
-	)
-	(zone
-		(net "Net-(U1-AC0)")
-		(layer "F.Cu")
-		(hatch none 0.1)
-		(priority 30000)
-		(attr
-			(teardrop
-				(type padvia)
-			)
-		)
-		(connect_pads yes
-			(clearance 0)
-		)
-		(min_thickness 0.0254)
-		(fill yes
-			(island_removal_mode 1)
-		)
-		(polygon
-			(pts
-				(xy 52.781062 81.915657) (xy 52.601457 82.095262) (xy 52.903429 82.429667) (xy 53.593518 82.907718)
-				(xy 53.115514 82.00545)
-			)
-		)
-	)
-	(zone
-		(net "Net-(U1-AC0)")
-		(layer "F.Cu")
-		(hatch none 0.1)
-		(priority 30003)
-		(attr
-			(teardrop
-				(type padvia)
-			)
-		)
-		(connect_pads yes
-			(clearance 0)
-		)
-		(min_thickness 0.0254)
-		(fill yes
-			(island_removal_mode 1)
-		)
-		(polygon
-			(pts
-				(xy 48.686632 78.6119) (xy 48.686632 78.4849) (xy 48.677627 78.489617) (xy 48.542462 78.352151)
-				(xy 48.266681 78.390314) (xy 48.234701 78.528086) (xy 48.629593 78.607183) (xy 48.65361 78.6119)
-			)
-		)
-	)
-	(zone
 		(layer "F.Cu")
 		(hatch edge 0.5)
@@
 			)
 		)
+	)
+	(zone
+		(net "Net-(U1-AC0)")
+		(layer "F.Cu")
+		(hatch none 0.1)
+		(priority 30000)
+		(attr
+			(teardrop
+				(type padvia)
+			)
+		)
+		(connect_pads yes
+			(clearance 0)
+		)
+		(min_thickness 0.0254)
+		(fill yes
+			(island_removal_mode 1)
+		)
+		(polygon
+			(pts
+				(xy 52.781062 81.915657) (xy 52.601457 82.095262) (xy 52.903429 82.429667) (xy 53.593518 82.907718)
+				(xy 53.115514 82.00545)
+			)
+		)
+	)
+	(zone
+		(net "Net-(U1-AC0)")
+		(layer "F.Cu")
+		(hatch none 0.1)
+		(priority 30001)
+		(attr
+			(teardrop
+				(type padvia)
+			)
+		)
+		(connect_pads yes
+			(clearance 0)
+		)
+		(min_thickness 0.0254)
+		(fill yes
+			(island_removal_mode 1)
+		)
+		(polygon
+			(pts
+				(xy 52.118353 81.612158) (xy 52.297958 81.432553) (xy 52.009499 81.107101) (xy 51.889251 81.203451)
+				(xy 51.941246 81.472044)
+			)
+		)
+	)
+	(zone
+		(net "Net-(U1-AC0)")
+		(layer "F.Cu")
+		(hatch none 0.1)
+		(priority 30003)
+		(attr
+			(teardrop
+				(type padvia)
+			)
+		)
+		(connect_pads yes
+			(clearance 0)
+		)
+		(min_thickness 0.0254)
+		(fill yes
+			(island_removal_mode 1)
+		)
+		(polygon
+			(pts
+				(xy 48.686632 78.6119) (xy 48.686632 78.4849) (xy 48.677627 78.489617) (xy 48.542462 78.352151)
+				(xy 48.266681 78.390314) (xy 48.234701 78.528086) (xy 48.629593 78.607183) (xy 48.65361 78.6119)
+			)
+		)
