File: PCB/uranus-pocket-tbc.kicad_sch (KiCad schematic)
At the start: 3 parts, among them U1 ST25DV04KC-IE8S3

Commit message: update schematic, oops
Other:
- note added: "-OR-"
- note removed: "OR"
- moved on the sheet: C2
Changed lines of the file:
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@@
 	(text "Inductance too high"
 		(exclude_from_sim no)
-		(at 142.24 112.522 0)
+		(at 142.24 113.792 0)
 		(effects
 			(font
@@
 		)
 	)
-	(text "OR"
+	(text "-OR-"
 		(exclude_from_sim no)
 		(at 144.526 108.458 0)
@@
 	(wire
 		(pts
-			(xy 129.54 121.92) (xy 129.54 127)
+			(xy 129.54 123.19) (xy 129.54 128.27)
 		)
 		(stroke
@@
 	(wire
 		(pts
-			(xy 135.89 129.54) (xy 135.89 120.65)
-		)
-		(stroke
-			(width 0)
-			(type default)
-		)
-	)
-	(wire
-		(pts
-			(xy 128.27 120.65) (xy 128.27 128.27)
+			(xy 135.89 130.81) (xy 135.89 121.92)
+		)
+		(stroke
+			(width 0)
+			(type default)
+		)
+	)
+	(wire
+		(pts
+			(xy 128.27 121.92) (xy 128.27 129.54)
 		)
 		(stroke
@@
 	(wire
 		(pts
-			(xy 138.43 118.11) (xy 125.73 118.11)
-		)
-		(stroke
-			(width 0)
-			(type default)
-		)
-	)
-	(wire
-		(pts
-			(xy 135.89 120.65) (xy 128.27 120.65)
+			(xy 138.43 119.38) (xy 125.73 119.38)
+		)
+		(stroke
+			(width 0)
+			(type default)
+		)
+	)
+	(wire
+		(pts
+			(xy 135.89 121.92) (xy 128.27 121.92)
 		)
 		(stroke
@@
 	(wire
 		(pts
-			(xy 125.73 130.81) (xy 137.16 130.81)
-		)
-		(stroke
-			(width 0)
-			(type default)
-		)
-	)
-	(wire
-		(pts
-			(xy 148.59 121.92) (xy 154.94 121.92)
-		)
-		(stroke
-			(width 0)
-			(type default)
-		)
-	)
-	(wire
-		(pts
-			(xy 137.16 119.38) (xy 127 119.38)
-		)
-		(stroke
-			(width 0)
-			(type default)
-		)
-	)
-	(wire
-		(pts
-			(xy 127 129.54) (xy 135.89 129.54)
+			(xy 125.73 132.08) (xy 137.16 132.08)
+		)
+		(stroke
+			(width 0)
+			(type default)
+		)
+	)
+	(wire
+		(pts
+			(xy 148.59 123.19) (xy 154.94 123.19)
+		)
+		(stroke
+			(width 0)
+			(type default)
+		)
+	)
+	(wire
+		(pts
+			(xy 137.16 120.65) (xy 127 120.65)
+		)
+		(stroke
+			(width 0)
+			(type default)
+		)
+	)
+	(wire
+		(pts
+			(xy 127 130.81) (xy 135.89 130.81)
 		)
 		(stroke
@@
 	(wire
 		(pts
-			(xy 129.54 127) (xy 154.94 127)
-		)
-		(stroke
-			(width 0)
-			(type default)
-		)
-	)
-	(wire
-		(pts
-			(xy 127 119.38) (xy 127 129.54)
+			(xy 129.54 128.27) (xy 154.94 128.27)
+		)
+		(stroke
+			(width 0)
+			(type default)
+		)
+	)
+	(wire
+		(pts
+			(xy 127 120.65) (xy 127 130.81)
 		)
 		(stroke
@@
 	(wire
 		(pts
-			(xy 137.16 130.81) (xy 137.16 119.38)
+			(xy 137.16 132.08) (xy 137.16 120.65)
 		)
 		(stroke
@@
 	(wire
 		(pts
-			(xy 128.27 128.27) (xy 134.62 128.27)
+			(xy 128.27 129.54) (xy 134.62 129.54)
 		)
 		(stroke
@@
 	(wire
 		(pts
-			(xy 134.62 121.92) (xy 129.54 121.92)
+			(xy 134.62 123.19) (xy 129.54 123.19)
 		)
 		(stroke
@@
 	(wire
 		(pts
-			(xy 125.73 118.11) (xy 125.73 130.81)
+			(xy 125.73 119.38) (xy 125.73 132.08)
 		)
 		(stroke
@@
 	(wire
 		(pts
-			(xy 138.43 121.92) (xy 143.51 121.92)
+			(xy 138.43 123.19) (xy 143.51 123.19)
 		)
 		(stroke
@@
 	(wire
 		(pts
-			(xy 138.43 121.92) (xy 138.43 118.11)
-		)
-		(stroke
-			(width 0)
-			(type default)
-		)
-	)
-	(wire
-		(pts
-			(xy 134.62 128.27) (xy 134.62 121.92)
+			(xy 138.43 123.19) (xy 138.43 119.38)
+		)
+		(stroke
+			(width 0)
+			(type default)
+		)
+	)
+	(wire
+		(pts
+			(xy 134.62 129.54) (xy 134.62 123.19)
 		)
 		(stroke
@@
 	(symbol
 		(lib_id "Device:C_Small")
-		(at 146.05 121.92 90)
+		(at 146.05 123.19 90)
 		(unit 1)
 		(body_style 1)
@@
 		(fields_autoplaced yes)
 		(property "Reference" "C2"
-			(at 146.05 115.57 90)
+			(at 146.05 116.84 90)
 			(show_name no)
 			(do_not_autoplace no)
@@
 		)
 		(property "Value" "tbd"
-			(at 146.05 118.11 90)
+			(at 146.05 119.38 90)
 			(show_name no)
 			(do_not_autoplace no)
@@
 		)
 		(property "Footprint" ""
-			(at 146.05 121.92 0)
+			(at 146.05 123.19 0)
 			(hide yes)
 			(show_name no)
@@
 		)
 		(property "Datasheet" ""
-			(at 146.05 121.92 0)
+			(at 146.05 123.19 0)
 			(hide yes)
 			(show_name no)
@@
 		)
 		(property "Description" "Unpolarized capacitor, small symbol"
-			(at 156.21 121.92 0)
+			(at 156.21 123.19 0)
 			(hide yes)
 			(show_name no)
